File: isolation.kicad_sch (KiCad schematic)
At the start: 48 parts, among them J2 NAPPE_FILAMENT_HT, U1 UCC27517, U12 UCC24612, U13 SN74LVC1G08, U3 ISO7710, U5 DPC817, U7 AMC0311R, U8 AMC0311R, U9 AMC0302R

Commit message: Retire la barriere d'isolation primaire/secondaire (secondaire non isole du primaire dans le montage final)
Decision utilisateur du 2026-10-25 : le secondaire de puissance (VOUT_N/
VOUT_P) ne sera plus flottant ni isole galvaniquement du primaire. La
regle .kicad_dru barriere_primaire_secondaire est retiree (commentee,
pas supprimee), la classe de nets SEC est conservee a titre
organisationnel dans KICAD-HT.kicad_pro. Seule la barriere controle
(C2000) <-> puissance reste une isolation reelle. 00-intention-conception.md,
README.md et doc/plan-isolation-4couches.md mis a jour (section 20bis).
Parts:
- removed C42: 10u, Capacitor_SMD:C_0805_2012Metric, symbol Device:C
- removed C43: 100n, Capacitor_SMD:C_0805_2012Metric, symbol Device:C
- removed R12: 1, Resistor_SMD:R_0805_2012Metric, symbol Device:R
- removed R35, R36, R40, R41, R42, R6: 1M, Resistor_SMD:R_0805_2012Metric, symbol Device:R
- removed U12: UCC24612, Package_TO_SOT_SMD:SOT-23-5, symbol custom_parts:UCC24612
