File: isolation.kicad_sch (KiCad schematic)
At the start: 38 parts, among them J2 NAPPE_FILAMENT_HT, U1 UCC27517, U13 SN74LVC1G08, U3 ISO7710, U5 DPC817, U7 AMC0311R, U8 AMC0311R, U9 AMC0302R

Commit message: Linearisation HV_BIAS : stabilise sous PWM reel (Rs=1k/Cint=100p), placement Q7
Le correctif precedent (Rs=330/Cint=1nF) n'avait ete valide qu'avec un
echelon analogique deja filtre, pas le vrai PWM du C2000. En rejouant la
boucle avec le PWM reel, elargir le filtre d'entree pour ecraser
l'ondulation residuelle (R47/Cin : 1k/1n -> 100k/100n) a reintroduit une
oscillation auto-entretenue differente (~700kHz), confirmee independante
du PWM via un echelon direct isole avant le filtre.

Nouveau correctif, verifie sur le profil complet de commande PWM (3,5s) :
Rs=1k (degenerescence Q6, au lieu de 330) + Cint=100pF (compensation
ampli-op, au lieu de 1nF) -- ondulation residuelle en sortie sous le mV.
Reporte sur polarisation.kicad_sch.

simulation/gen_pwm_breakpoints.py : genere la table PWL explicite
necessaire pour que LTspice resolve correctement les impulsions PWM
etroites -- une expression comportementale IF(TIME...) ne declare aucun
breakpoint, le solveur en sautait ~98% sans elle.

Cote PCB : placement de l'empreinte Q7 (BSS127I, SOT-23) sur la feuille
Polarisation ; isolation.kicad_sch renomme NAPPE_FILAMENT_HT -> DC_HT.

Co-Authored-By: Claude Sonnet 5 <noreply@anthropic.com>
Parts:
- J2: value NAPPE_FILAMENT_HT -> DC_HT
Changed lines of the file:
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@@
 			)
 		)
-		(property "Value" "NAPPE_FILAMENT_HT"
+		(property "Value" "DC_HT"
 			(at 399.288 190.5 0)
 			(show_name no)

Commit message: Routage en cours : retouches schema (alim/flyback/isolation/limitation-courant/polarisation), doc renommage Temp_ht->I_Out_ht et NAPPE_FILAMENT_HT->DC_HT, fix .kicad_dru (commentaires #), nettoyage simulation/results
Co-Authored-By: Claude Sonnet 5 <noreply@anthropic.com>
Parts:
- removed C25, C26: 100n, Capacitor_SMD:C_0805_2012Metric, symbol Device:C
- removed C29: 100p, Capacitor_SMD:C_0805_2012Metric, symbol Device:C
- removed C30: 1n, Capacitor_SMD:C_0805_2012Metric, symbol Device:C
- removed R16: 10k, Resistor_SMD:R_0805_2012Metric, symbol Device:R
- removed R17: 100, Resistor_SMD:R_0805_2012Metric, symbol Device:R
- removed TH1: 10k_B4000, Resistor_SMD:R_0805_2012Metric, symbol Device:Thermistor_NTC
- removed U8: AMC0311R, SOIC_DWV:SOIC-8_DWV_5.85x11.5mm_P1.27mm, symbol custom_parts:AMC0311R
- added C37, C49: 100n, Capacitor_SMD:C_0805_2012Metric, symbol Device:C
- added C60: 47n, Capacitor_SMD:C_0805_2012Metric, symbol Device:C
- added C63, C67: 10n, Capacitor_SMD:C_0805_2012Metric, symbol Device:C
- added C64, C65, C66, C68: 1n, Capacitor_SMD:C_0805_2012Metric, symbol Device:C
- added R26: 1k, Resistor_SMD:R_0805_2012Metric, symbol Device:R
- added R40, R41, R42, R43: 10, Resistor_SMD:R_0805_2012Metric, symbol Device:R
- added U22: AMC0302R, SOIC_DWV:SOIC-8_DWV_5.85x11.5mm_P1.27mm, symbol custom_parts:AMC0302R
Connections:
- net 3V3_ISO: now also C49.1, U22.8 (VDD2)
- net GND: now also C66.2, C68.2
- net GND_CTRL: now also C49.2, C60.2, U22.5 (GND2), U22.6 (REFIN)
- net ISNS_KN: now also R43.1; no longer U9.3 (INN)
- net ISNS_KP: now also R42.1; no longer U9.2 (INP)
- net RAIL_3V3_SEC: now also C37.1, U22.1 (VDD1)
- net VOUT_N: now also C37.2, C64.2, C65.2, R41.1, U22.4 (GND1)
- net Temp_ht renamed I_Out_ht
- net I_Out_ht: now also C60.1, R26.2
- new net: C63.2, C65.1, R41.2, U22.3 (INN)
- new net: C67.1, C68.1, R42.2, U9.2 (INP)
- new net: C66.1, C67.2, R43.2, U9.3 (INN)
- new net: R26.1, U22.7 (OUT)
- new net: C63.1, C64.1, R40.2, U22.2 (INP)
- new net ISNS_P: R40.1
Other:
- moved on the sheet: C31, C32, C33, C46, R18, U9

Commit message: Corrige le sliver VOUT_N/GND, remet les trous de fixation, fixe le 3D de F1
Travail de nettoyage silkscreen (texte titre, champs reference, J2) et
contour de zone (pointe de cuivre VOUT_N pres du via RAIL_8V25, decouverte
via reconstruction geometrique des zones remplies faute de coordonnees
dans le rapport DRC). Modele 3D de F1 repointe vers
Fuseholder_Cylinder-5x20mm_Schurter_0031_8201_Horizontal_Open.step
(echelle 0.836 pour coller au pas 18.8mm existant) -- le fichier original
Littelfuse_111_Lateral n'a jamais existe dans la bibliotheque 3D KiCad
stock (verifie sur le depot officiel), aucune pastille ni routage touche.

DRC propre (0 violation).

Co-Authored-By: Claude Sonnet 5 <noreply@anthropic.com>
Parts:
- removed R37, R38, R39: 1M, Resistor_SMD:R_0805_2012Metric, symbol Device:R

Commit message: Ajoute Q8/U5 (driver optocoupleur PWM_EN) et classe Net-(Q8-D) en CTRL
Q8 (MMBF170, NMOS) pilote U5 (DPC817) pour ne pas charger le
microcontroleur sur PWM_EN. Le net Net-(Q8-D) (drain Q8 <-> cathode U5)
tombait hors de la netclasse CTRL par defaut, declenchant 14 violations
barriere_controle contre ses voisins CTRL (R3, C34, U10, R37) pourtant
dans le meme sous-circuit. Verifie par tracage (Q8 gate=PWM_EN,
source=GND_CTRL ; U5 anode via R3=3V3_ISO) avant classement, comme pour
les ajouts precedents a SEC. DRC : 14 erreurs -> 0.

Documente aussi le fix du retour de masse J2 (§30, remove_unused_layers
sur les 10 broches signal).

Co-Authored-By: Claude Sonnet 5 <noreply@anthropic.com>
Parts:
- added Q8: MMBF170, Package_TO_SOT_SMD:SOT-23, symbol Transistor_FET:Q_NMOS_GSD
- added R37: 100k, Resistor_SMD:R_0805_2012Metric, symbol Device:R
Connections:
- net 3V3_ISO: now also R3.1
- net GND_CTRL: now also Q8.2 (S), R37.2; no longer U5.2
- net PWM_EN: now also Q8.1 (G), R37.1; no longer R3.1
- new net: Q8.3 (D), U5.2
