File: polarisation.kicad_sch (KiCad schematic)
At the start: 21 parts, among them J1 HV80_IN, Q3 BSS127I, Q4 MMBT2222, Q5 BSS127I, U10 ISO7710, U11 AMC0311R

Commit message: Retire la barriere d'isolation primaire/secondaire (secondaire non isole du primaire dans le montage final)
Decision utilisateur du 2026-10-25 : le secondaire de puissance (VOUT_N/
VOUT_P) ne sera plus flottant ni isole galvaniquement du primaire. La
regle .kicad_dru barriere_primaire_secondaire est retiree (commentee,
pas supprimee), la classe de nets SEC est conservee a titre
organisationnel dans KICAD-HT.kicad_pro. Seule la barriere controle
(C2000) <-> puissance reste une isolation reelle. 00-intention-conception.md,
README.md et doc/plan-isolation-4couches.md mis a jour (section 20bis).
Parts:
- added C27: 100n, Capacitor_SMD:C_0805_2012Metric, symbol Device:C
- added R40, R41, R42: 1M, Resistor_SMD:R_0805_2012Metric, symbol Device:R
Connections:
- net GND: now also C27.2, R42.1
- net HV_BIAS: now also C27.1, R40.2
- new net: R40.1, R41.2
- new net: R41.1, R42.2
Other:
- moved on the sheet: R20
