File: flyback.kicad_sch (KiCad schematic)
At the start: 20 parts, among them Q1 IPD050N10N5, Q2 IPD050N10N5, T1 MSD1514-103ME, U12 UCC24612

Commit message: Routage en cours : retouches schema (alim/flyback/isolation/limitation-courant/polarisation), doc renommage Temp_ht->I_Out_ht et NAPPE_FILAMENT_HT->DC_HT, fix .kicad_dru (commentaires #), nettoyage simulation/results
Co-Authored-By: Claude Sonnet 5 <noreply@anthropic.com>
Parts:
- added Q4: MMBF170, Package_TO_SOT_SMD:SOT-23, symbol Transistor_FET:Q_NMOS_GSD
- added Q5: IPD60R360P7, TO252:TO252-3_TabPin2, symbol custom_parts:MOSFET_3PIN_TAB2_TO252
- added R21: 100k, Resistor_SMD:R_0805_2012Metric, symbol Device:R
- added R25: 10m, Resistor_SMD:R_1210_3225Metric_Pad1.30x2.65mm_HandSolder, symbol Device:R
- added R35: 150, Resistor_SMD:R_0805_2012Metric, symbol Device:R
- added U20: VODA1275, VODA1275:SMD-4_VODA1275_VIS, symbol custom_parts:VODA1275
Connections:
- net VOUT_N: now also R25.1; no longer Out1.2 (Pin_2)
- net VOUT_P: now also Q5.2 (D); no longer Out1.1 (Pin_1)
- net HV_BIAS renamed HV_BIAS_OUT
- new net: R35.2, U20.1 (A)
- new net 3V3_ISO: R35.1
- new net GND_CTRL: Q4.2 (S), R21.2
- new net ISNS_P: Out1.2 (Pin_2), R25.2
- new net Q5_LED_K: Q4.3 (D), U20.2 (K)
- new net U15_OUTP: Q5.1 (G), U20.4 (OUT+)
- new net V_HT_OUT: Out1.1 (Pin_1), Q5.3 (S), U20.3 (OUT-)
- new net Vht_EN: Q4.1 (G), R21.1
Other:
- moved on the sheet: D4, Q2, R8
