File: alim.kicad_sch (KiCad schematic)
At the start: 13 parts

Commit message: Corrige le sliver VOUT_N/GND, remet les trous de fixation, fixe le 3D de F1
Travail de nettoyage silkscreen (texte titre, champs reference, J2) et
contour de zone (pointe de cuivre VOUT_N pres du via RAIL_8V25, decouverte
via reconstruction geometrique des zones remplies faute de coordonnees
dans le rapport DRC). Modele 3D de F1 repointe vers
Fuseholder_Cylinder-5x20mm_Schurter_0031_8201_Horizontal_Open.step
(echelle 0.836 pour coller au pas 18.8mm existant) -- le fichier original
Littelfuse_111_Lateral n'a jamais existe dans la bibliotheque 3D KiCad
stock (verifie sur le depot officiel), aucune pastille ni routage touche.

DRC propre (0 violation).

Co-Authored-By: Claude Sonnet 5 <noreply@anthropic.com>
Parts:
- added H1, H2, H3, H4: MountingScrew, MountingHole:MountingHole_3.2mm_M3, symbol Auxiliary_Items:MountingScrew

Commit message: Dissipation Reg1/Reg2, vias Q1 ajustes, retouches TVS
- Reg1 (LM317M) et Reg2 (MCP1703-3302) : connexion solide (zone_connect
  solid) sur les pastilles sortie/masse ; petite surface de dissipation
  RAIL_3V3_PRI sur B.Cu sous Reg2.
- Q1 : 18->12 vias thermiques, 6 retirees car elles barraient le passage
  de la zone RAIL_8V25 sur In2.Cu. Impact thermique verifie negligeable
  a la dissipation reelle de Q1 (~0,7W, simulation), encore confortable
  au cas pessimiste 2,1W/50degC (toutes pertes dans Q1, Rth(j-c) Infineon
  IPD050N10N5 = 1K/W max, Tj max 175degC).
- Via VOUT_N repositionne (143.87/87.61) pour stitcher F.Cu<->In1.Cu sans
  chevaucher la pastille du condensateur voisin ni les zones GND(B.Cu)/
  RAIL_3V3_PRI(In2.Cu).
- D3/D5/D8 (TVS) : SMCJ*->SMBJ* (boitier D_SMC->D_SMB).

DRC : 0 erreur (3 avertissements lib_footprint_mismatch bénins connus).

Co-Authored-By: Claude Sonnet 5 <noreply@anthropic.com>
Parts:
- D2: value SMCJ10A -> SMBJ9; footprint Diode_SMD:D_SMC -> Diode_SMD:D_SMB
- D7: value SMCJ04A -> SMBJ05; footprint Diode_SMD:D_SMC -> Diode_SMD:D_SMB
Changed lines of the file:
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@@
 			)
 		)
-		(property "Value" "SMCJ04A"
+		(property "Value" "SMBJ05"
 			(at 176.784 105.918 90)
 			(show_name no)
@@
 			)
 		)
-		(property "Footprint" "Diode_SMD:D_SMC"
+		(property "Footprint" "Diode_SMD:D_SMB"
 			(at 169.672 106.934 0)
 			(hide yes)
@@
 			)
 		)
-		(property "Value" "SMCJ10A"
+		(property "Value" "SMBJ9"
 			(at 97.282 118.11 90)
 			(show_name no)
@@
 			)
 		)
-		(property "Footprint" "Diode_SMD:D_SMC"
+		(property "Footprint" "Diode_SMD:D_SMB"
 			(at 90.17 119.126 0)
 			(hide yes)
